Commit message: add colision and foot

File: install/bot_desc/share/bot_desc/urdf/mybot/actor/caster.urdf.xacro (robot description, xacro)
@@ -13,4 +13,13 @@
                 </material>
             </visual>
+            <collision>
+                <origin xyz="0.0 0.0 0.0" rpy="0.0 0.0 0.0"/>
+                <geometry>
+                    <sphere radius="0.016"/>
+                </geometry>
+                <material name="yellow">
+                    <color rgba="1.0 1.0 0.0 0.8"/>
+                </material>
+            </collision>
         </link>
         <!--连接身体和轮子的关节-->

File: install/bot_desc/share/bot_desc/urdf/mybot/actor/wheel.urdf.xacro (robot description, xacro)
@@ -13,4 +13,13 @@
                 </material>
             </visual>
+            <collision>
+                <origin xyz="0.0 0.0 0.0" rpy="1.57079 0.0 0.0"/>
+                <geometry>
+                    <cylinder radius="0.032" length="0.04"/>
+                </geometry>
+                <material name="yellow">
+                    <color rgba="1.0 1.0 0.0 0.8"/>
+                </material>
+            </collision>
         </link>
         <!--连接身体和轮子的关节-->

File: install/bot_desc/share/bot_desc/urdf/mybot/base.urdf.xacro (robot description, xacro)
@@ -2,4 +2,5 @@
 <robot xmlns:xacro="http://www.ros.org/wiki/xacro">
     <xacro:macro name ="base_xacro" params="length radius">
+        <link name="base_footprint" />
         <!--机器人的身体部分-->
         <link name="base_link">
@@ -16,5 +17,21 @@
                 </material>
             </visual>
+            <collision>
+                <origin xyz="0.0 0.0 0.0" rpy="0.0 0.0 0.0"/>
+                    <!--几何形状-->
+                    <geometry>
+                        <cylinder radius="${radius}" length="${length}"/>
+                    </geometry>
+                    <!--材质和颜色描述-->
+                    <material name="white">
+                        <color rgba="1.0 1.0 1.0 0.5"/>
+                    </material>
+            </collision>
         </link>
+        <joint name="joint_name" type="fixed">
+            <parent link="base_footprint"/>
+            <child link="base_link"/>
+            <origin xyz="0.0 0.0 ${length/2.0 + 0.032-0.001}" rpy="0.0 0.0 0.0"/>
+        </joint>
     </xacro:macro>
 </robot>

File: install/bot_desc/share/bot_desc/urdf/mybot/labot.urdf.xacro (robot description, xacro)
@@ -18,6 +18,6 @@
     <xacro:imu_xacro xyz="0.10 0.0 0.075"/>
     <xacro:camera_xacro xyz="0.0 0.0 0.1"/>
-    <xacro:wheel_xacro wheel_name="left_wheel" xyz="0.1 0.1 -0.06"/>
-    <xacro:wheel_xacro wheel_name="right_wheel" xyz="0.1 -0.1 -0.06"/>
+    <xacro:wheel_xacro wheel_name="left_wheel" xyz="0 0.1 -0.06"/>
+    <xacro:wheel_xacro wheel_name="right_wheel" xyz="0 -0.1 -0.06"/>
     <xacro:caster_xacro caster_name="front_caster" xyz="0.08 0.0 -0.076"/>
     <xacro:caster_xacro caster_name="rear_caster" xyz="0.08 -0.0 -0.076"/>

File: install/bot_desc/share/bot_desc/urdf/mybot/sensor/camera.urdf.xacro (robot description, xacro)
@@ -13,4 +13,13 @@
                 </material>
             </visual>
+            <collision>
+                <origin xyz="0.0 0.0 0.0" rpy="0.0 0.0 0.0"/>
+                <geometry>
+                    <box size="0.02 0.02 0.02"/>
+                </geometry>
+                <material name="green">
+                    <color rgba="0.0 1.0 0.0 0.5"/>
+                </material>
+            </collision>
         </link>
         <!--连接身体和相机的关节-->

File: install/bot_desc/share/bot_desc/urdf/mybot/sensor/imu.urdf.xacro (robot description, xacro)
@@ -13,4 +13,13 @@
                 </material>
             </visual>
+            <collision>
+                <origin xyz="0.0 0.0 0.0" rpy="0.0 0.0 0.0"/>
+                <geometry>
+                    <box size="0.02 0.02 0.02"/>
+                </geometry>
+                <material name="blue">
+                    <color rgba="0.0 0.0 1.0 0.5"/>
+                </material>
+            </collision>
         </link>
         <!--连接身体和IMU的关节-->

File: install/bot_desc/share/bot_desc/urdf/mybot/sensor/laser.urdf.xacro (robot description, xacro)
@@ -13,4 +13,13 @@
                 </material>
             </visual>
+            <collision>
+                <origin xyz="0.0 0.0 0.0" rpy="0.0 0.0 0.0"/>
+                <geometry>
+                    <cylinder radius="0.01" length="0.1"/>
+                </geometry>
+                <material name="gray">
+                    <color rgba="0.5 0.5 0.5 1.0"/>
+                </material>
+            </collision>
         </link>
          <!--机器人的激光雷达部件-->
@@ -25,4 +34,13 @@
                 </material>
             </visual>
+            <collision>
+                <origin xyz="0.0 0.0 0.0" rpy="0.0 0.0 0.0"/>
+                <geometry>
+                    <cylinder radius="0.02" length="0.2"/>
+                </geometry>
+                <material name="red">
+                    <color rgba="1.0 0.0 0.0 0.5"/>
+                </material>
+            </collision>
         </link>
         <!--连接身体和激光雷达的关节-->

Commit message: ros2 launch bot_desc gazebo_sim.launch.py 加载机器人模型并add gazebo 标签

File: install/bot_desc/share/bot_desc/urdf/mybot/actor/caster.urdf.xacro (robot description, xacro)
@@ -31,4 +31,11 @@
             <origin xyz="${xyz}" rpy="0.0 0.0 0.0"/>
         </joint>
+        <gazebo reference="${caster_name}_link">
+            <mu1 value="0.0"/>
+            <mu2 value="0.0"/>
+            <kp value="1000000000.0"/>
+            <kd value="1.0"/>
+            <material>Gazebo/Yellow</material>
+        </gazebo>
     </xacro:macro>
 </robot>

File: install/bot_desc/share/bot_desc/urdf/mybot/actor/wheel.urdf.xacro (robot description, xacro)
@@ -32,4 +32,11 @@
             <axis xyz="0.0 1.0 0.0"/>
         </joint>
+            <gazebo reference="${wheel_name}_link">
+                <mu1 value="20.0"/>
+                <mu2 value="20.0"/>
+                <kp value="1000000000.0"/>
+                <kd value="1.0"/>
+                <material>Gazebo/Yellow</material>
+            </gazebo>
     </xacro:macro>
 </robot>

File: install/bot_desc/share/bot_desc/urdf/mybot/sensor/imu.urdf.xacro (robot description, xacro)
@@ -31,4 +31,7 @@
             <origin xyz="${xyz}" rpy="0.0 0.0 0.0"/>
         </joint>
+            <gazebo reference="imu_link">
+                <material>Gazebo/Blue</material>
+            </gazebo>
     </xacro:macro>
 </robot>

File: install/bot_desc/share/bot_desc/urdf/mybot/sensor/laser.urdf.xacro (robot description, xacro)
@@ -58,4 +58,10 @@
             <origin xyz="${xyz}" rpy="0.0 0.0 0.0"/>
         </joint>
+        <gazebo reference="laser_cylinder_link">
+            <material>Gazebo/Black</material>
+        </gazebo>
+        <gazebo reference="laser_link">
+            <material>Gazebo/Black</material>
+        </gazebo>
     </xacro:macro>
 </robot>

Commit message: add imu and camera sim

File: install/bot_desc/share/bot_desc/urdf/mybot/actor/caster.urdf.xacro (robot description, xacro)
@@ -1,41 +1 @@
-<?xml version="1.0"?>
-<robot xmlns:xacro="http://www.ros.org/wiki/xacro">
-    <xacro:include filename="$(find bot_desc)/urdf/mybot/common_inertia.xacro"/>
-    <xacro:macro name ="caster_xacro" params="caster_name xyz">
-         <!--机器人的轮子部件-->
-        <link name="${caster_name}_link">
-            <visual>
-                <origin xyz="0.0 0.0 0.0" rpy="0.0 0.0 0.0"/>
-                <geometry>
-                    <sphere radius="0.016"/>
-                </geometry>
-                <material name="yellow">
-                    <color rgba="1.0 1.0 0.0 0.8"/>
-                </material>
-            </visual>
-            <collision>
-                <origin xyz="0.0 0.0 0.0" rpy="0.0 0.0 0.0"/>
-                <geometry>
-                    <sphere radius="0.016"/>
-                </geometry>
-                <material name="yellow">
-                    <color rgba="1.0 1.0 0.0 0.8"/>
-                </material>
-            </collision>
-            <xacro:sphere_inertia m="0.05" r="0.016"/>
-        </link>
-        <!--连接身体和轮子的关节-->
-        <joint name="${caster_name}_joint" type="fixed">
-            <parent link="base_link"/>
-            <child link="${caster_name}_link"/>
-            <origin xyz="${xyz}" rpy="0.0 0.0 0.0"/>
-        </joint>
-        <gazebo reference="${caster_name}_link">
-            <mu1 value="0.0"/>
-            <mu2 value="0.0"/>
-            <kp value="1000000000.0"/>
-            <kd value="1.0"/>
-            <material>Gazebo/Yellow</material>
-        </gazebo>
-    </xacro:macro>
-</robot>
+/home/jungle/ros_cpp/robot-/src/bot_desc/urdf/mybot/actor/caster.urdf.xacro

File: install/bot_desc/share/bot_desc/urdf/mybot/actor/wheel.urdf.xacro (robot description, xacro)
@@ -1,42 +1 @@
-<?xml version="1.0"?>
-<robot xmlns:xacro="http://www.ros.org/wiki/xacro">
-    <xacro:include filename="$(find bot_desc)/urdf/mybot/common_inertia.xacro"/>
-    <xacro:macro name ="wheel_xacro" params="wheel_name xyz">
-         <!--机器人的轮子部件-->
-        <link name="${wheel_name}_link">
-            <visual>
-                <origin xyz="0.0 0.0 0.0" rpy="1.57079 0.0 0.0"/>
-                <geometry>
-                    <cylinder radius="0.032" length="0.04"/>
-                </geometry>
-                <material name="yellow">
-                    <color rgba="1.0 1.0 0.0 0.8"/>
-                </material>
-            </visual>
-            <collision>
-                <origin xyz="0.0 0.0 0.0" rpy="1.57079 0.0 0.0"/>
-                <geometry>
-                    <cylinder radius="0.032" length="0.04"/>
-                </geometry>
-                <material name="yellow">
-                    <color rgba="1.0 1.0 0.0 0.8"/>
-                </material>
-            </collision>
-            <xacro:cylinder_inertia m="0.05" r="0.032" h="0.04"/>
-        </link>
-        <!--连接身体和轮子的关节-->
-        <joint name="${wheel_name}_joint" type="continuous">
-            <parent link="base_link"/>
-            <child link="${wheel_name}_link"/>
-            <origin xyz="${xyz}" rpy="0.0 0.0 0.0"/>
-            <axis xyz="0.0 1.0 0.0"/>
-        </joint>
-            <gazebo reference="${wheel_name}_link">
-                <mu1 value="20.0"/>
-                <mu2 value="20.0"/>
-                <kp value="1000000000.0"/>
-                <kd value="1.0"/>
-                <material>Gazebo/Yellow</material>
-            </gazebo>
-    </xacro:macro>
-</robot>
+/home/jungle/ros_cpp/robot-/src/bot_desc/urdf/mybot/actor/wheel.urdf.xacro

File: install/bot_desc/share/bot_desc/urdf/mybot/base.urdf.xacro (robot description, xacro)
@@ -1,40 +1 @@
-<?xml version="1.0"?>
-<robot xmlns:xacro="http://www.ros.org/wiki/xacro">
-    <xacro:include filename="$(find bot_desc)/urdf/mybot/common_inertia.xacro"/>
-    <xacro:macro name ="base_xacro" params="length radius">
-        <link name="base_footprint" />
-        <!--机器人的身体部分-->
-        <link name="base_link">
-        <!--部件的外观描述-->
-            <visual>
-                <origin xyz="0.0 0.0 0.0" rpy="0.0 0.0 0.0"/>
-                <!--几何形状-->
-                <geometry>
-                    <cylinder radius="${radius}" length="${length}"/>
-                </geometry>
-                <!--材质和颜色描述-->
-                <material name="white">
-                    <color rgba="1.0 1.0 1.0 0.5"/>
-                </material>
-            </visual>
-            <collision>
-                <origin xyz="0.0 0.0 0.0" rpy="0.0 0.0 0.0"/>
-                    <!--几何形状-->
-                    <geometry>
-                        <cylinder radius="${radius}" length="${length}"/>
-                    </geometry>
-                    <!--材质和颜色描述-->
-                    <material name="white">
-                        <color rgba="1.0 1.0 1.0 0.5"/>
-                    </material>
-            </collision>
-            <!--部件的惯性描述-->
-            <xacro:cylinder_inertia m="2.0" r="${radius}" h="${length}"/>
-        </link>
-        <joint name="joint_name" type="fixed">
-            <parent link="base_footprint"/>
-            <child link="base_link"/>
-            <origin xyz="0.0 0.0 ${length/2.0 + 0.032-0.001}" rpy="0.0 0.0 0.0"/>
-        </joint>
-    </xacro:macro>
-</robot>
+/home/jungle/ros_cpp/robot-/src/bot_desc/urdf/mybot/base.urdf.xacro

File: install/bot_desc/share/bot_desc/urdf/mybot/common_inertia.xacro (robot description, xacro)
@@ -1,23 +1 @@
-<?xml version="1.0"?>
-<robot xmlns:xacro="http://www.ros.org/wiki/xacro">
-    <xacro:macro name="box_inertia" params="m w h d">
-        <inertial>
-            <origin xyz="0 0 0" rpy="0 0 0"/>
-            <mass value="${m}"/>
-            <inertia ixx="${m / 12*(h*h+d*d)}" ixy="0" ixz="0" iyy="${m / 12*(w*w+d*d)}" iyz="0" izz="${m / 12*(w*w+h*h)}"/>
-        </inertial>
-    </xacro:macro>
-    <xacro:macro name="cylinder_inertia" params="m r h">
-        <inertial>
-            <origin xyz="0 0 0" rpy="0 0 0"/>
-            <mass value="${m}"/>
-            <inertia ixx="${m / 12*(h*h+3*r*r)}" ixy="0" ixz="0" iyy="${m / 12*(3*r*r+h*h)}" iyz="0" izz="${m / 2*(r*r)}"/>
-        </inertial>
-    </xacro:macro>
-    <xacro:macro name="sphere_inertia" params="m r">
-        <inertial>
-            <origin xyz="0 0 0" rpy="0 0 0"/>
-            <mass value="${m}"/>
-            <inertia ixx="${(2/5)*m*(r*r)}" ixy="0" ixz="0" iyy="${(2/5)*m*(r*r)}" iyz="0" izz="${(2/5)*m*(r*r)}"/>
-        </inertial>
-    </xacro:macro></robot>
+/home/jungle/ros_cpp/robot-/src/bot_desc/urdf/mybot/common_inertia.xacro

File: install/bot_desc/share/bot_desc/urdf/mybot/labot.urdf.xacro (robot description, xacro)
@@ -1,27 +1 @@
-<?xml version="1.0"?>
-<robot xmlns:xacro="http://www.ros.org/wiki/xacro" name="labot">
-    <!--包含身体部件的xacro文件-->
-    <xacro:include filename="$(find bot_desc)/urdf/mybot/base.urdf.xacro"/>
-    <!--包含激光雷达部件的xacro文件-->
-    <xacro:include filename="$(find bot_desc)/urdf/mybot/sensor/laser.urdf.xacro"/>
-    <!--包含IMU部件的xacro文件-->
-    <xacro:include filename="$(find bot_desc)/urdf/mybot/sensor/imu.urdf.xacro"/>
-    <!--包含相机部件的xacro文件-->
-    <xacro:include filename="$(find bot_desc)/urdf/mybot/sensor/camera.urdf.xacro"/>
-    <!--包含轮子部件的xacro文件-->
-    <xacro:include filename="$(find bot_desc)/urdf/mybot/actor/wheel.urdf.xacro"/>
-    <!--包含万向轮部件的xacro文件-->
-    <xacro:include filename="$(find bot_desc)/urdf/mybot/actor/caster.urdf.xacro"/>
-    <!--插件-->
-    <xacro:include filename="$(find bot_desc)/urdf/mybot/plugins/gazebo_control_plugin.xacro"/>
-    <!--使用宏来实例化身体和传感器部件，并设置它们的位置参数-->
-    <xacro:base_xacro length="0.12" radius="0.1"/>
-    <xacro:laser_xacro xyz="0.0 0.0 0.10"/>
-    <xacro:imu_xacro xyz="0.0 0.0 0.02"/>
-    <xacro:camera_xacro xyz="0.1 0.0 0.075"/>
-    <xacro:wheel_xacro wheel_name="left_wheel" xyz="0 0.1 -0.06"/>
-    <xacro:wheel_xacro wheel_name="right_wheel" xyz="0 -0.1 -0.06"/>
-    <xacro:caster_xacro caster_name="front_caster" xyz="0.08 0.0 -0.076"/>
-    <xacro:caster_xacro caster_name="rear_caster" xyz="-0.08 0.0 -0.076"/>
-    <xacro:gazebo_control_plugin />
-</robot>
+/home/jungle/ros_cpp/robot-/src/bot_desc/urdf/mybot/labot.urdf.xacro

File: install/bot_desc/share/bot_desc/urdf/mybot/plugins/gazebo_control_plugin.xacro (robot description, xacro)
@@ -1,27 +1 @@
-<?xml version ="1.0"?>
-<robot xmlns:xacro="http://www.ros.org/wiki/xacro">
-    <xacro:macro name="gazebo_control_plugin">
-        <gazebo>
-            <plugin name="diff_drive" filename="libgazebo_ros_diff_drive.so">
-                <ros>
-                    <namespace>/</namespace>
-                    <remapping>cmd_vel:=cmd_vel</remapping>
-                    <remapping>odom:=odom</remapping>
-                </ros>
-                <update_rate>30.0</update_rate>
-                <!--wheel-->
-                <left_joint>left_wheel_joint</left_joint>
-                <right_joint>right_wheel_joint</right_joint>
-                <wheel_separation>0.2</wheel_separation>
-                <wheel_diameter>0.064</wheel_diameter>
-                <max_wheel_torque>20.0</max_wheel_torque>
-                <max_wheel_acceleration>10.0</max_wheel_acceleration>
-                <publish_odom>true</publish_odom>
-                <publish_odom_tf>true</publish_odom_tf>
-                <publish_wheel_tf>true</publish_wheel_tf>
-                <odometry_frame>odom</odometry_frame>
-                <robot_base_frame>base_footprint</robot_base_frame>
-            </plugin>
-        </gazebo>
-    </xacro:macro>
-</robot>
+/home/jungle/ros_cpp/robot-/src/bot_desc/urdf/mybot/plugins/gazebo_control_plugin.xacro

File: install/bot_desc/share/bot_desc/urdf/mybot/sensor/camera.urdf.xacro (robot description, xacro)
@@ -1,34 +1 @@
-<?xml version="1.0"?>
-<robot xmlns:xacro="http://www.ros.org/wiki/xacro">
-    <xacro:include filename="$(find bot_desc)/urdf/mybot/common_inertia.xacro"/>
-    <xacro:macro name ="camera_xacro" params="xyz">
-         <!--机器人的相机部件-->
-        <link name="camera_link">
-            <visual>
-                <origin xyz="0.0 0.0 0.0" rpy="0.0 0.0 0.0"/>
-                <geometry>
-                    <box size="0.02 0.02 0.02"/>
-                </geometry>
-                <material name="green">
-                    <color rgba="0.0 1.0 0.0 0.5"/>
-                </material>
-            </visual>
-            <collision>
-                <origin xyz="0.0 0.0 0.0" rpy="0.0 0.0 0.0"/>
-                <geometry>
-                    <box size="0.02 0.02 0.02"/>
-                </geometry>
-                <material name="green">
-                    <color rgba="0.0 1.0 0.0 0.5"/>
-                </material>
-            </collision>
-            <xacro:box_inertia m="0.1" d="0.02" w="0.02" h="0.02"/>
-        </link>
-        <!--连接身体和相机的关节-->
-        <joint name="camera_joint" type="fixed">
-            <parent link="base_link"/>
-            <child link="camera_link"/>
-            <origin xyz="${xyz}" rpy="0.0 0.0 0.0"/>
-        </joint>
-    </xacro:macro>
-</robot>
+/home/jungle/ros_cpp/robot-/src/bot_desc/urdf/mybot/sensor/camera.urdf.xacro

File: install/bot_desc/share/bot_desc/urdf/mybot/sensor/imu.urdf.xacro (robot description, xacro)
@@ -1,37 +1 @@
-<?xml version="1.0"?>
-<robot xmlns:xacro="http://www.ros.org/wiki/xacro">
-    <xacro:include filename="$(find bot_desc)/urdf/mybot/common_inertia.xacro"/>
-    <xacro:macro name ="imu_xacro" params="xyz">
-         <!--机器人的IMU部件，惯性测量传感器-->
-        <link name="imu_link">
-            <visual>
-                <origin xyz="0.0 0.0 0.0" rpy="0.0 0.0 0.0"/>
-                <geometry>
-                    <box size="0.02 0.02 0.02"/>
-                </geometry>
-                <material name="blue">
-                    <color rgba="0.0 0.0 1.0 0.5"/>
-                </material>
-            </visual>
-            <collision>
-                <origin xyz="0.0 0.0 0.0" rpy="0.0 0.0 0.0"/>
-                <geometry>
-                    <box size="0.02 0.02 0.02"/>
-                </geometry>
-                <material name="blue">
-                    <color rgba="0.0 0.0 1.0 0.5"/>
-                </material>
-            </collision>
-            <xacro:box_inertia m="0.05" w="0.02" h="0.02" d="0.02"/>
-        </link>
-        <!--连接身体和IMU的关节-->
-        <joint name="imu_joint" type="fixed">
-            <parent link="base_link"/>
-            <child link="imu_link"/>
-            <origin xyz="${xyz}" rpy="0.0 0.0 0.0"/>
-        </joint>
-            <gazebo reference="imu_link">
-                <material>Gazebo/Blue</material>
-            </gazebo>
-    </xacro:macro>
-</robot>
+/home/jungle/ros_cpp/robot-/src/bot_desc/urdf/mybot/sensor/imu.urdf.xacro

File: install/bot_desc/share/bot_desc/urdf/mybot/sensor/laser.urdf.xacro (robot description, xacro)
@@ -1,67 +1 @@
-<?xml version="1.0"?>
-<robot xmlns:xacro="http://www.ros.org/wiki/xacro">
-    <xacro:include filename="$(find bot_desc)/urdf/mybot/common_inertia.xacro"/>
-    <xacro:macro name ="laser_xacro" params="xyz">
-    <!--雷达支撑杆-->
-        <link name="laser_cylinder_link">
-            <visual>
-                <origin xyz="0.0 0.0 0.0" rpy="0.0 0.0 0.0"/>
-                <geometry>
-                    <cylinder radius="0.01" length="0.1"/>
-                </geometry>
-                <material name="gray">
-                    <color rgba="0.5 0.5 0.5 1.0"/>
-                </material>
-            </visual>
-            <collision>
-                <origin xyz="0.0 0.0 0.0" rpy="0.0 0.0 0.0"/>
-                <geometry>
-                    <cylinder radius="0.01" length="0.1"/>
-                </geometry>
-                <material name="gray">
-                    <color rgba="0.5 0.5 0.5 1.0"/>
-                </material>
-            </collision>
-            <xacro:cylinder_inertia m="0.05" r="0.01" h="0.1"/>
-        </link>
-         <!--机器人的激光雷达部件-->
-        <link name="laser_link">
-            <visual>
-                <origin xyz="0.0 0.0 0.0" rpy="0.0 0.0 0.0"/>
-                <geometry>
-                    <cylinder radius="0.02" length="0.02"/>
-                </geometry>
-                <material name="red">
-                    <color rgba="1.0 0.0 0.0 0.5"/>
-                </material>
-            </visual>
-            <collision>
-                <origin xyz="0.0 0.0 0.0" rpy="0.0 0.0 0.0"/>
-                <geometry>
-                    <cylinder radius="0.02" length="0.02"/>
-                </geometry>
-                <material name="red">
-                    <color rgba="1.0 0.0 0.0 0.5"/>
-                </material>
-            </collision>
-            <xacro:cylinder_inertia m="0.1" r="0.02" h="0.02"/>
-        </link>
-        <!--连接身体和激光雷达的关节-->
-        <joint name="laser_joint" type="fixed">
-            <parent link="laser_cylinder_link"/>
-            <child link="laser_link"/>
-            <origin xyz="0.0 0.0 0.05" rpy="0.0 0.0 0.0"/>
-        </joint>
-        <joint name="laser_cylinder_joint" type="fixed">
-            <parent link="base_link"/>
-            <child link="laser_cylinder_link"/>
-            <origin xyz="${xyz}" rpy="0.0 0.0 0.0"/>
-        </joint>
-        <gazebo reference="laser_cylinder_link">
-            <material>Gazebo/Black</material>
-        </gazebo>
-        <gazebo reference="laser_link">
-            <material>Gazebo/Black</material>
-        </gazebo>
-    </xacro:macro>
-</robot>
+/home/jungle/ros_cpp/robot-/src/bot_desc/urdf/mybot/sensor/laser.urdf.xacro

File: src/bot_desc/urdf/mybot/labot.urdf.xacro (robot description, xacro)
@@ -15,4 +15,5 @@
     <!--插件-->
     <xacro:include filename="$(find bot_desc)/urdf/mybot/plugins/gazebo_control_plugin.xacro"/>
+    <xacro:include filename="$(find bot_desc)/urdf/mybot/plugins/gazebo_sensor_plugin.xacro"/>
     <!--使用宏来实例化身体和传感器部件，并设置它们的位置参数-->
     <xacro:base_xacro length="0.12" radius="0.1"/>
@@ -25,3 +26,4 @@
     <xacro:caster_xacro caster_name="rear_caster" xyz="-0.08 0.0 -0.076"/>
     <xacro:gazebo_control_plugin />
+    <xacro:gazebo_sensor_plugin />
 </robot>
