Commit message: add imu and camera sim

File: src/bot_desc/urdf/mybot/plugins/gazebo_sensor_plugin.xacro (robot description, xacro)
@@ -1,26 +1,141 @@
 <?xml version ="1.0"?>
 <robot xmlns:xacro="http://www.ros.org/wiki/xacro">
+    <!--激光雷达传感器仿真-->
     <xacro:macro name="gazebo_sensor_plugin">
-        <gazebo>
-            <plugin name="laser_plugin" filename="libgazebo_ros_laser.so">
-                <ros>
-                    <namespace>/</namespace>
-                    <remapping>scan:=scan</remapping>
-                </ros>
-            </plugin>
-            <plugin name="imu_plugin" filename="libgazebo_ros_imu.so">
-                <ros>
-                    <namespace>/</namespace>
-                    <remapping>imu:=imu</remapping>
-                </ros>
-            </plugin>
-            <plugin name="camera_plugin" filename="libgazebo_ros_camera.so">
-                <ros>
-                    <namespace>/</namespace>
-                    <remapping>image:=image</remapping>
-                    <remapping>camera_info:=camera_info</remapping>
-                </ros>
-            </plugin>
+        <gazebo reference="laser_link">
+            <sensor name="laserscan" type="ray">
+                <!--设置插件参数-->
+                <plugin name="laserscan" filename="libgazebo_ros_ray_sensor.so">
+                    <ros>
+                        <namespace>/</namespace>
+                        <remapping>~/out:=scan</remapping>
+                    </ros>
+                    <output_type>sensor_msgs/LaserScan</output_type>
+                    <frame_name>laser_link</frame_name>
+                </plugin>
+                <always_on>true</always_on>
+                <visualize>true</visualize>
+                <update_rate>5.0</update_rate>
+                <pose>0 0 0 0 0 0</pose>
+                <!--设置扫描参数-->
+                <ray>
+                    <scan>
+                    <!--设置扫描范围-->
+                        <horizontal>
+                            <samples>360</samples>
+                            <resolution>1</resolution>
+                            <min_angle>0</min_angle>
+                            <max_angle>6.28</max_angle>
+                        </horizontal>
+                    </scan>
+                    <!--设置扫描距离-->
+                    <range>
+                        <min>0.12</min>
+                        <max>8</max>
+                        <resolution>0.015</resolution>
+                    </range>
+                    <!--设置噪声-->
+                    <noise type="gaussian">
+                        <mean>0.0</mean>
+                        <stddev>0.01</stddev>
+                    </noise>
+                </ray>
+            </sensor>
         </gazebo>
+        <!--惯性测量单元仿真-->
+            <gazebo reference="imu_link">
+                <sensor name="imu_sensor" type="imu">
+                    <plugin name="imu_plugin" filename="libgazebo_ros_imu_sensor.so">
+                        <ros>
+                            <namespace>/</namespace>
+                            <remapping>~/out:=imu</remapping>
+                        </ros>
+                        <initial_orientation_as_reference>false</initial_orientation_as_reference>
+                    </plugin>
+                    <always_on>true</always_on>
+                    <update_rate>100.0</update_rate>
+                    <!--六轴噪声设置-->
+                    <imu>
+                        <angular_velocity>
+                            <x>
+                                <noise type="gaussian">
+                                    <mean>0.0</mean>
+                                    <stddev>2e-4</stddev>
+                                    <bias_mean>0.0000075</bias_mean>
+                                    <bias_stddev>0.0000008</bias_stddev>
+                                </noise>
+                            </x>
+                            <y>
+                                <noise type="gaussian">
+                                    <mean>0.0</mean>
+                                    <stddev>2e-4</stddev>
+                                    <bias_mean>0.0000075</bias_mean>
+                                    <bias_stddev>0.0000008</bias_stddev>
+                                </noise>
+                            </y>
+                            <z>
+                                <noise type="gaussian">
+                                    <mean>0.0</mean>
+                                    <stddev>2e-4</stddev>
+                                    <bias_mean>0.0000075</bias_mean>
+                                    <bias_stddev>0.0000008</bias_stddev>
+                                </noise>
+                            </z>
+                        </angular_velocity>
+                        <linear_acceleration>
+                            <x>
+                                <noise type="gaussian">
+                                    <mean>0.0</mean>
+                                    <stddev>2e-4</stddev>
+                                    <bias_mean>0.0000075</bias_mean>
+                                    <bias_stddev>0.0000008</bias_stddev>
+                                </noise>
+                            </x>
+                            <y>
+                                <noise type="gaussian">
+                                    <mean>0.0</mean>
+                                    <stddev>2e-4</stddev>
+                                    <bias_mean>0.0000075</bias_mean>
+                                    <bias_stddev>0.0000008</bias_stddev>
+                                </noise>
+                            </y>
+                            <z>
+                                <noise type="gaussian">
+                                    <mean>0.0</mean>
+                                    <stddev>2e-4</stddev>
+                                    <bias_mean>0.0000075</bias_mean>
+                                    <bias_stddev>0.0000008</bias_stddev>
+                                </noise>
+                            </z>
+                        </linear_acceleration>
+                    </imu>
+                </sensor>
+            </gazebo>
+            <!--相机仿真-->
+            <gazebo reference="camera_link">
+                <sensor name="camera_sensor" type="depth">
+                    <plugin name="depth_camera" filename="libgazebo_ros_camera.so">
+                        <frame_name>camera_optical_link</frame_name>
+                    </plugin>
+                    <always_on>true</always_on>
+                    <update_rate>10.0</update_rate>
+                    <camera name="camera">
+                        <horizontal_fov>1.5009831567</horizontal_fov>
+                        <image>
+                            <width>800</width>
+                            <height>600</height>
+                            <format>R8G8B8</format>
+                        </image>
+                        <distortion>
+                            <k1>0</k1>
+                            <k2>0</k2>
+                            <k3>0</k3>
+                            <p1>0</p1>
+                            <p2>0</p2>
+                            <center>0.5 0.5</center>
+                        </distortion>
+                    </camera>
+                </sensor>
+            </gazebo>
     </xacro:macro>
 </robot>

File: src/bot_desc/urdf/mybot/sensor/camera.urdf.xacro (robot description, xacro)
@@ -25,4 +25,5 @@
             <xacro:box_inertia m="0.1" d="0.02" w="0.02" h="0.02"/>
         </link>
+        <link name="camera_optical_link"> </link>
         <!--连接身体和相机的关节-->
         <joint name="camera_joint" type="fixed">
@@ -31,4 +32,9 @@
             <origin xyz="${xyz}" rpy="0.0 0.0 0.0"/>
         </joint>
+        <joint name="camera_optical_joint" type="fixed">
+            <parent link="camera_link"/>
+            <child link="camera_optical_link"/>
+            <origin xyz="0 0 0" rpy="${-pi/2} 0 ${-pi/2}"/>
+        </joint>
     </xacro:macro>
 </robot>
