Commit message: complete inertia and study gazebo

File: install/bot_desc/share/bot_desc/urdf/first_robot.xacro (robot description, xacro)
@@ -1 +1,43 @@
-/home/jungle/ros_cpp/robot-/src/bot_desc/urdf/first_robot.xacro
+<?xml version="1.0"?>
+<robot xmlns:xacro="http://www.ros.org/wiki/xacro" name="first_robot">
+    <xacro:macro name ="base_link" params="length radius">
+        <!--机器人的身体部分-->
+        <link name="base_link">
+        <!--部件的外观描述-->
+            <visual>
+                <origin xyz="0.0 0.0 0.0" rpy="0.0 0.0 0.0"/>
+                <!--几何形状-->
+                <geometry>
+                    <cylinder radius="${radius}" length="${length}"/>
+                </geometry>
+                <!--材质和颜色描述-->
+                <material name="white">
+                    <color rgba="1.0 1.0 1.0 0.5"/>
+                </material>
+            </visual>
+        </link>
+    </xacro:macro>
+    <xacro:macro name ="imu_link" params="imu_name xyz">
+         <!--机器人的IMU部件，惯性测量传感器-->
+        <link name="${imu_name}_link">
+            <visual>
+                <origin xyz="0.0 0.0 0.0" rpy="0.0 0.0 0.0"/>
+                <geometry>
+                    <box size="0.02 0.02 0.02"/>
+                </geometry>
+                <material name="blue">
+                    <color rgba="0.0 0.0 1.0 0.5"/>
+                </material>
+            </visual>
+        </link>
+        <!--连接身体和IMU的关节-->
+        <joint name="${imu_name}_joint" type="fixed">
+            <parent link="base_link"/>
+            <child link="${imu_name}_link"/>
+            <origin xyz="${xyz}" rpy="0.0 0.0 0.0"/>
+        </joint>
+    </xacro:macro>
+    <xacro:base_link length="0.2" radius="0.1"/>
+    <xacro:imu_link imu_name="imu_up" xyz="0.0 0.0 0.03"/>
+    <xacro:imu_link imu_name="imu_down" xyz="0.0 0.0 -0.03"/>
+</robot>

File: install/bot_desc/share/bot_desc/urdf/mybot/actor/caster.urdf.xacro (robot description, xacro)
@@ -1 +1,34 @@
-/home/jungle/ros_cpp/robot-/src/bot_desc/urdf/mybot/actor/caster.urdf.xacro
+<?xml version="1.0"?>
+<robot xmlns:xacro="http://www.ros.org/wiki/xacro">
+    <xacro:include filename="$(find bot_desc)/urdf/mybot/common_inertia.xacro"/>
+    <xacro:macro name ="caster_xacro" params="caster_name xyz">
+         <!--机器人的轮子部件-->
+        <link name="${caster_name}_link">
+            <visual>
+                <origin xyz="0.0 0.0 0.0" rpy="0.0 0.0 0.0"/>
+                <geometry>
+                    <sphere radius="0.016"/>
+                </geometry>
+                <material name="yellow">
+                    <color rgba="1.0 1.0 0.0 0.8"/>
+                </material>
+            </visual>
+            <collision>
+                <origin xyz="0.0 0.0 0.0" rpy="0.0 0.0 0.0"/>
+                <geometry>
+                    <sphere radius="0.016"/>
+                </geometry>
+                <material name="yellow">
+                    <color rgba="1.0 1.0 0.0 0.8"/>
+                </material>
+            </collision>
+            <xacro:sphere_inertia m="0.05" r="0.016"/>
+        </link>
+        <!--连接身体和轮子的关节-->
+        <joint name="${caster_name}_joint" type="fixed">
+            <parent link="base_link"/>
+            <child link="${caster_name}_link"/>
+            <origin xyz="${xyz}" rpy="0.0 0.0 0.0"/>
+        </joint>
+    </xacro:macro>
+</robot>

File: install/bot_desc/share/bot_desc/urdf/mybot/actor/wheel.urdf.xacro (robot description, xacro)
@@ -1 +1,35 @@
-/home/jungle/ros_cpp/robot-/src/bot_desc/urdf/mybot/actor/wheel.urdf.xacro
+<?xml version="1.0"?>
+<robot xmlns:xacro="http://www.ros.org/wiki/xacro">
+    <xacro:include filename="$(find bot_desc)/urdf/mybot/common_inertia.xacro"/>
+    <xacro:macro name ="wheel_xacro" params="wheel_name xyz">
+         <!--机器人的轮子部件-->
+        <link name="${wheel_name}_link">
+            <visual>
+                <origin xyz="0.0 0.0 0.0" rpy="1.57079 0.0 0.0"/>
+                <geometry>
+                    <cylinder radius="0.032" length="0.04"/>
+                </geometry>
+                <material name="yellow">
+                    <color rgba="1.0 1.0 0.0 0.8"/>
+                </material>
+            </visual>
+            <collision>
+                <origin xyz="0.0 0.0 0.0" rpy="1.57079 0.0 0.0"/>
+                <geometry>
+                    <cylinder radius="0.032" length="0.04"/>
+                </geometry>
+                <material name="yellow">
+                    <color rgba="1.0 1.0 0.0 0.8"/>
+                </material>
+            </collision>
+            <xacro:cylinder_inertia m="0.05" r="0.032" h="0.04"/>
+        </link>
+        <!--连接身体和轮子的关节-->
+        <joint name="${wheel_name}_joint" type="continuous">
+            <parent link="base_link"/>
+            <child link="${wheel_name}_link"/>
+            <origin xyz="${xyz}" rpy="0.0 0.0 0.0"/>
+            <axis xyz="0.0 1.0 0.0"/>
+        </joint>
+    </xacro:macro>
+</robot>

File: install/bot_desc/share/bot_desc/urdf/mybot/base.urdf.xacro (robot description, xacro)
@@ -1 +1,40 @@
-/home/jungle/ros_cpp/robot-/src/bot_desc/urdf/mybot/base.urdf.xacro
+<?xml version="1.0"?>
+<robot xmlns:xacro="http://www.ros.org/wiki/xacro">
+    <xacro:include filename="$(find bot_desc)/urdf/mybot/common_inertia.xacro"/>
+    <xacro:macro name ="base_xacro" params="length radius">
+        <link name="base_footprint" />
+        <!--机器人的身体部分-->
+        <link name="base_link">
+        <!--部件的外观描述-->
+            <visual>
+                <origin xyz="0.0 0.0 0.0" rpy="0.0 0.0 0.0"/>
+                <!--几何形状-->
+                <geometry>
+                    <cylinder radius="${radius}" length="${length}"/>
+                </geometry>
+                <!--材质和颜色描述-->
+                <material name="white">
+                    <color rgba="1.0 1.0 1.0 0.5"/>
+                </material>
+            </visual>
+            <collision>
+                <origin xyz="0.0 0.0 0.0" rpy="0.0 0.0 0.0"/>
+                    <!--几何形状-->
+                    <geometry>
+                        <cylinder radius="${radius}" length="${length}"/>
+                    </geometry>
+                    <!--材质和颜色描述-->
+                    <material name="white">
+                        <color rgba="1.0 1.0 1.0 0.5"/>
+                    </material>
+            </collision>
+            <!--部件的惯性描述-->
+            <xacro:cylinder_inertia m="1.0" r="${radius}" h="${length}"/>
+        </link>
+        <joint name="joint_name" type="fixed">
+            <parent link="base_footprint"/>
+            <child link="base_link"/>
+            <origin xyz="0.0 0.0 ${length/2.0 + 0.032-0.001}" rpy="0.0 0.0 0.0"/>
+        </joint>
+    </xacro:macro>
+</robot>

File: install/bot_desc/share/bot_desc/urdf/mybot/labot.urdf.xacro (robot description, xacro)
@@ -1 +1,24 @@
-/home/jungle/ros_cpp/robot-/src/bot_desc/urdf/mybot/labot.urdf.xacro
+<?xml version="1.0"?>
+<robot xmlns:xacro="http://www.ros.org/wiki/xacro" name="labot">
+    <!--包含身体部件的xacro文件-->
+    <xacro:include filename="$(find bot_desc)/urdf/mybot/base.urdf.xacro"/>
+    <!--包含激光雷达部件的xacro文件-->
+    <xacro:include filename="$(find bot_desc)/urdf/mybot/sensor/laser.urdf.xacro"/>
+    <!--包含IMU部件的xacro文件-->
+    <xacro:include filename="$(find bot_desc)/urdf/mybot/sensor/imu.urdf.xacro"/>
+    <!--包含相机部件的xacro文件-->
+    <xacro:include filename="$(find bot_desc)/urdf/mybot/sensor/camera.urdf.xacro"/>
+    <!--包含轮子部件的xacro文件-->
+    <xacro:include filename="$(find bot_desc)/urdf/mybot/actor/wheel.urdf.xacro"/>
+    <!--包含万向轮部件的xacro文件-->
+    <xacro:include filename="$(find bot_desc)/urdf/mybot/actor/caster.urdf.xacro"/>
+    <!--使用宏来实例化身体和传感器部件，并设置它们的位置参数-->
+    <xacro:base_xacro length="0.12" radius="0.1"/>
+    <xacro:laser_xacro xyz="0.0 0.0 0.10"/>
+    <xacro:imu_xacro xyz="0.0 0.0 0.02"/>
+    <xacro:camera_xacro xyz="0.1 0.0 0.075"/>
+    <xacro:wheel_xacro wheel_name="left_wheel" xyz="0 0.1 -0.06"/>
+    <xacro:wheel_xacro wheel_name="right_wheel" xyz="0 -0.1 -0.06"/>
+    <xacro:caster_xacro caster_name="front_caster" xyz="0.08 0.0 -0.076"/>
+    <xacro:caster_xacro caster_name="rear_caster" xyz="-0.08 0.0 -0.076"/>
+</robot>

File: install/bot_desc/share/bot_desc/urdf/mybot/sensor/camera.urdf.xacro (robot description, xacro)
@@ -1 +1,34 @@
-/home/jungle/ros_cpp/robot-/src/bot_desc/urdf/mybot/sensor/camera.urdf.xacro
+<?xml version="1.0"?>
+<robot xmlns:xacro="http://www.ros.org/wiki/xacro">
+    <xacro:include filename="$(find bot_desc)/urdf/mybot/common_inertia.xacro"/>
+    <xacro:macro name ="camera_xacro" params="xyz">
+         <!--机器人的相机部件-->
+        <link name="camera_link">
+            <visual>
+                <origin xyz="0.0 0.0 0.0" rpy="0.0 0.0 0.0"/>
+                <geometry>
+                    <box size="0.02 0.02 0.02"/>
+                </geometry>
+                <material name="green">
+                    <color rgba="0.0 1.0 0.0 0.5"/>
+                </material>
+            </visual>
+            <collision>
+                <origin xyz="0.0 0.0 0.0" rpy="0.0 0.0 0.0"/>
+                <geometry>
+                    <box size="0.02 0.02 0.02"/>
+                </geometry>
+                <material name="green">
+                    <color rgba="0.0 1.0 0.0 0.5"/>
+                </material>
+            </collision>
+            <xacro:box_inertia m="0.1" d="0.02" w="0.02" h="0.02"/>
+        </link>
+        <!--连接身体和相机的关节-->
+        <joint name="camera_joint" type="fixed">
+            <parent link="base_link"/>
+            <child link="camera_link"/>
+            <origin xyz="${xyz}" rpy="0.0 0.0 0.0"/>
+        </joint>
+    </xacro:macro>
+</robot>

File: install/bot_desc/share/bot_desc/urdf/mybot/sensor/imu.urdf.xacro (robot description, xacro)
@@ -1 +1,34 @@
-/home/jungle/ros_cpp/robot-/src/bot_desc/urdf/mybot/sensor/imu.urdf.xacro
+<?xml version="1.0"?>
+<robot xmlns:xacro="http://www.ros.org/wiki/xacro">
+    <xacro:include filename="$(find bot_desc)/urdf/mybot/common_inertia.xacro"/>
+    <xacro:macro name ="imu_xacro" params="xyz">
+         <!--机器人的IMU部件，惯性测量传感器-->
+        <link name="imu_link">
+            <visual>
+                <origin xyz="0.0 0.0 0.0" rpy="0.0 0.0 0.0"/>
+                <geometry>
+                    <box size="0.02 0.02 0.02"/>
+                </geometry>
+                <material name="blue">
+                    <color rgba="0.0 0.0 1.0 0.5"/>
+                </material>
+            </visual>
+            <collision>
+                <origin xyz="0.0 0.0 0.0" rpy="0.0 0.0 0.0"/>
+                <geometry>
+                    <box size="0.02 0.02 0.02"/>
+                </geometry>
+                <material name="blue">
+                    <color rgba="0.0 0.0 1.0 0.5"/>
+                </material>
+            </collision>
+            <xacro:box_inertia m="0.05" w="0.02" h="0.02" d="0.02"/>
+        </link>
+        <!--连接身体和IMU的关节-->
+        <joint name="imu_joint" type="fixed">
+            <parent link="base_link"/>
+            <child link="imu_link"/>
+            <origin xyz="${xyz}" rpy="0.0 0.0 0.0"/>
+        </joint>
+    </xacro:macro>
+</robot>

File: install/bot_desc/share/bot_desc/urdf/mybot/sensor/laser.urdf.xacro (robot description, xacro)
@@ -1 +1,61 @@
-/home/jungle/ros_cpp/robot-/src/bot_desc/urdf/mybot/sensor/laser.urdf.xacro
+<?xml version="1.0"?>
+<robot xmlns:xacro="http://www.ros.org/wiki/xacro">
+    <xacro:include filename="$(find bot_desc)/urdf/mybot/common_inertia.xacro"/>
+    <xacro:macro name ="laser_xacro" params="xyz">
+    <!--雷达支撑杆-->
+        <link name="laser_cylinder_link">
+            <visual>
+                <origin xyz="0.0 0.0 0.0" rpy="0.0 0.0 0.0"/>
+                <geometry>
+                    <cylinder radius="0.01" length="0.1"/>
+                </geometry>
+                <material name="gray">
+                    <color rgba="0.5 0.5 0.5 1.0"/>
+                </material>
+            </visual>
+            <collision>
+                <origin xyz="0.0 0.0 0.0" rpy="0.0 0.0 0.0"/>
+                <geometry>
+                    <cylinder radius="0.01" length="0.1"/>
+                </geometry>
+                <material name="gray">
+                    <color rgba="0.5 0.5 0.5 1.0"/>
+                </material>
+            </collision>
+            <xacro:cylinder_inertia m="0.05" r="0.01" h="0.1"/>
+        </link>
+         <!--机器人的激光雷达部件-->
+        <link name="laser_link">
+            <visual>
+                <origin xyz="0.0 0.0 0.0" rpy="0.0 0.0 0.0"/>
+                <geometry>
+                    <cylinder radius="0.02" length="0.02"/>
+                </geometry>
+                <material name="red">
+                    <color rgba="1.0 0.0 0.0 0.5"/>
+                </material>
+            </visual>
+            <collision>
+                <origin xyz="0.0 0.0 0.0" rpy="0.0 0.0 0.0"/>
+                <geometry>
+                    <cylinder radius="0.02" length="0.02"/>
+                </geometry>
+                <material name="red">
+                    <color rgba="1.0 0.0 0.0 0.5"/>
+                </material>
+            </collision>
+            <xacro:cylinder_inertia m="0.1" r="0.02" h="0.02"/>
+        </link>
+        <!--连接身体和激光雷达的关节-->
+        <joint name="laser_joint" type="fixed">
+            <parent link="laser_cylinder_link"/>
+            <child link="laser_link"/>
+            <origin xyz="0.0 0.0 0.05" rpy="0.0 0.0 0.0"/>
+        </joint>
+        <joint name="laser_cylinder_joint" type="fixed">
+            <parent link="base_link"/>
+            <child link="laser_cylinder_link"/>
+            <origin xyz="${xyz}" rpy="0.0 0.0 0.0"/>
+        </joint>
+    </xacro:macro>
+</robot>

File: src/bot_desc/urdf/mybot/actor/caster.urdf.xacro (robot description, xacro)
@@ -23,4 +23,5 @@
                 </material>
             </collision>
+            <xacro:sphere_inertia m="0.05" r="0.016"/>
         </link>
         <!--连接身体和轮子的关节-->

File: src/bot_desc/urdf/mybot/actor/wheel.urdf.xacro (robot description, xacro)
@@ -23,4 +23,5 @@
                 </material>
             </collision>
+            <xacro:cylinder_inertia m="0.05" r="0.032" h="0.04"/>
         </link>
         <!--连接身体和轮子的关节-->

File: src/bot_desc/urdf/mybot/labot.urdf.xacro (robot description, xacro)
@@ -15,10 +15,10 @@
     <!--使用宏来实例化身体和传感器部件，并设置它们的位置参数-->
     <xacro:base_xacro length="0.12" radius="0.1"/>
-    <xacro:laser_xacro xyz="0.0 0.0 0.02"/>
-    <xacro:imu_xacro xyz="0.10 0.0 0.075"/>
-    <xacro:camera_xacro xyz="0.0 0.0 0.1"/>
+    <xacro:laser_xacro xyz="0.0 0.0 0.10"/>
+    <xacro:imu_xacro xyz="0.0 0.0 0.02"/>
+    <xacro:camera_xacro xyz="0.1 0.0 0.075"/>
     <xacro:wheel_xacro wheel_name="left_wheel" xyz="0 0.1 -0.06"/>
     <xacro:wheel_xacro wheel_name="right_wheel" xyz="0 -0.1 -0.06"/>
     <xacro:caster_xacro caster_name="front_caster" xyz="0.08 0.0 -0.076"/>
-    <xacro:caster_xacro caster_name="rear_caster" xyz="0.08 -0.0 -0.076"/>
+    <xacro:caster_xacro caster_name="rear_caster" xyz="-0.08 0.0 -0.076"/>
 </robot>

File: src/bot_desc/urdf/mybot/sensor/camera.urdf.xacro (robot description, xacro)
@@ -23,4 +23,5 @@
                 </material>
             </collision>
+            <xacro:box_inertia m="0.1" d="0.02" w="0.02" h="0.02"/>
         </link>
         <!--连接身体和相机的关节-->

File: src/bot_desc/urdf/mybot/sensor/imu.urdf.xacro (robot description, xacro)
@@ -23,4 +23,5 @@
                 </material>
             </collision>
+            <xacro:box_inertia m="0.05" w="0.02" h="0.02" d="0.02"/>
         </link>
         <!--连接身体和IMU的关节-->

File: src/bot_desc/urdf/mybot/sensor/laser.urdf.xacro (robot description, xacro)
@@ -23,4 +23,5 @@
                 </material>
             </collision>
+            <xacro:cylinder_inertia m="0.05" r="0.01" h="0.1"/>
         </link>
          <!--机器人的激光雷达部件-->
@@ -29,5 +30,5 @@
                 <origin xyz="0.0 0.0 0.0" rpy="0.0 0.0 0.0"/>
                 <geometry>
-                    <cylinder radius="0.02" length="0.2"/>
+                    <cylinder radius="0.02" length="0.02"/>
                 </geometry>
                 <material name="red">
@@ -38,5 +39,5 @@
                 <origin xyz="0.0 0.0 0.0" rpy="0.0 0.0 0.0"/>
                 <geometry>
-                    <cylinder radius="0.02" length="0.2"/>
+                    <cylinder radius="0.02" length="0.02"/>
                 </geometry>
                 <material name="red">
@@ -44,4 +45,5 @@
                 </material>
             </collision>
+            <xacro:cylinder_inertia m="0.1" r="0.02" h="0.02"/>
         </link>
         <!--连接身体和激光雷达的关节-->
