Commit message: have bug no fix

File: install/bot_desc/share/bot_desc/urdf/mybot/sensor/imu.urdf.xacro (robot description, xacro)
@@ -1,37 +1 @@
-<?xml version="1.0"?>
-<robot xmlns:xacro="http://www.ros.org/wiki/xacro">
-    <xacro:include filename="$(find bot_desc)/urdf/mybot/common_inertia.xacro"/>
-    <xacro:macro name ="imu_xacro" params="xyz">
-         <!--机器人的IMU部件，惯性测量传感器-->
-        <link name="imu_link">
-            <visual>
-                <origin xyz="0.0 0.0 0.0" rpy="0.0 0.0 0.0"/>
-                <geometry>
-                    <box size="0.02 0.02 0.02"/>
-                </geometry>
-                <material name="blue">
-                    <color rgba="0.0 0.0 1.0 0.5"/>
-                </material>
-            </visual>
-            <collision>
-                <origin xyz="0.0 0.0 0.0" rpy="0.0 0.0 0.0"/>
-                <geometry>
-                    <box size="0.02 0.02 0.02"/>
-                </geometry>
-                <material name="blue">
-                    <color rgba="0.0 0.0 1.0 0.5"/>
-                </material>
-            </collision>
-            <xacro:box_inertia m="0.05" w="0.02" h="0.02" d="0.02"/>
-        </link>
-        <!--连接身体和IMU的关节-->
-        <joint name="imu_joint" type="fixed">
-            <parent link="base_link"/>
-            <child link="imu_link"/>
-            <origin xyz="${xyz}" rpy="0.0 0.0 0.0"/>
-        </joint>
-            <gazebo reference="imu_link">
-                <material>Gazebo/Blue</material>
-            </gazebo>
-    </xacro:macro>
-</robot>
+/home/jungle/ros_cpp/robot-/robot-/src/bot_desc/urdf/mybot/sensor/imu.urdf.xacro

File: install/bot_desc/share/bot_desc/urdf/mybot/sensor/laser.urdf.xacro (robot description, xacro)
@@ -1,67 +1 @@
-<?xml version="1.0"?>
-<robot xmlns:xacro="http://www.ros.org/wiki/xacro">
-    <xacro:include filename="$(find bot_desc)/urdf/mybot/common_inertia.xacro"/>
-    <xacro:macro name ="laser_xacro" params="xyz">
-    <!--雷达支撑杆-->
-        <link name="laser_cylinder_link">
-            <visual>
-                <origin xyz="0.0 0.0 0.0" rpy="0.0 0.0 0.0"/>
-                <geometry>
-                    <cylinder radius="0.01" length="0.1"/>
-                </geometry>
-                <material name="gray">
-                    <color rgba="0.5 0.5 0.5 1.0"/>
-                </material>
-            </visual>
-            <collision>
-                <origin xyz="0.0 0.0 0.0" rpy="0.0 0.0 0.0"/>
-                <geometry>
-                    <cylinder radius="0.01" length="0.1"/>
-                </geometry>
-                <material name="gray">
-                    <color rgba="0.5 0.5 0.5 1.0"/>
-                </material>
-            </collision>
-            <xacro:cylinder_inertia m="0.05" r="0.01" h="0.1"/>
-        </link>
-         <!--机器人的激光雷达部件-->
-        <link name="laser_link">
-            <visual>
-                <origin xyz="0.0 0.0 0.0" rpy="0.0 0.0 0.0"/>
-                <geometry>
-                    <cylinder radius="0.02" length="0.02"/>
-                </geometry>
-                <material name="red">
-                    <color rgba="1.0 0.0 0.0 0.5"/>
-                </material>
-            </visual>
-            <collision>
-                <origin xyz="0.0 0.0 0.0" rpy="0.0 0.0 0.0"/>
-                <geometry>
-                    <cylinder radius="0.02" length="0.02"/>
-                </geometry>
-                <material name="red">
-                    <color rgba="1.0 0.0 0.0 0.5"/>
-                </material>
-            </collision>
-            <xacro:cylinder_inertia m="0.1" r="0.02" h="0.02"/>
-        </link>
-        <!--连接身体和激光雷达的关节-->
-        <joint name="laser_joint" type="fixed">
-            <parent link="laser_cylinder_link"/>
-            <child link="laser_link"/>
-            <origin xyz="0.0 0.0 0.05" rpy="0.0 0.0 0.0"/>
-        </joint>
-        <joint name="laser_cylinder_joint" type="fixed">
-            <parent link="base_link"/>
-            <child link="laser_cylinder_link"/>
-            <origin xyz="${xyz}" rpy="0.0 0.0 0.0"/>
-        </joint>
-        <gazebo reference="laser_cylinder_link">
-            <material>Gazebo/Black</material>
-        </gazebo>
-        <gazebo reference="laser_link">
-            <material>Gazebo/Black</material>
-        </gazebo>
-    </xacro:macro>
-</robot>
+/home/jungle/ros_cpp/robot-/robot-/src/bot_desc/urdf/mybot/sensor/laser.urdf.xacro

File: src/bot_desc/urdf/mybot/labot.urdf.xacro (robot description, xacro)
@@ -14,7 +14,8 @@
     <xacro:include filename="$(find bot_desc)/urdf/mybot/actor/caster.urdf.xacro"/>
     <!--插件-->
+    <xacro:include filename="$(find bot_desc)/urdf/mybot/plugins/gazebo_sensor_plugin.xacro"/>
     <xacro:include filename="$(find bot_desc)/urdf/mybot/mybot_ros2_control.xacro"/>
-    <xacro:include filename="$(find bot_desc)/urdf/mybot/plugins/gazebo_sensor_plugin.xacro"/>
-    <!--使用宏来实例化身体和传感器部件，并设置它们的位置参数-->
+    <xacro:include filename="$(find bot_desc)/urdf/mybot/plugins/gazebo_control_plugin.xacro"/>
+    <!--使用宏来实例化身体和传感器部件并设置它们的位置参数-->
     <xacro:base_xacro length="0.12" radius="0.1"/>
     <xacro:laser_xacro xyz="0.0 0.0 0.10"/>
@@ -25,5 +26,5 @@
     <xacro:caster_xacro caster_name="front_caster" xyz="0.08 0.0 -0.076"/>
     <xacro:caster_xacro caster_name="rear_caster" xyz="-0.08 0.0 -0.076"/>
+    <xacro:gazebo_sensor_plugin />
     <xacro:mybot_ros2_control />
-    <xacro:gazebo_sensor_plugin />
 </robot>

File: src/bot_desc/urdf/mybot/sensor/imu.urdf.xacro (robot description, xacro)
@@ -3,5 +3,5 @@
     <xacro:include filename="$(find bot_desc)/urdf/mybot/common_inertia.xacro"/>
     <xacro:macro name ="imu_xacro" params="xyz">
-         <!--机器人的IMU部件，惯性测量传感器-->
+         <!--机器人的IMU部件and惯性测量传感器-->
         <link name="imu_link">
             <visual>
