Commit message: fix bug

File: install/bot_desc/share/bot_desc/urdf/mybot/sensor/imu.urdf.xacro (robot description, xacro)
@@ -1 +1,37 @@
-/home/jungle/ros_cpp/robot-/robot-/src/bot_desc/urdf/mybot/sensor/imu.urdf.xacro
+<?xml version="1.0"?>
+<robot xmlns:xacro="http://www.ros.org/wiki/xacro">
+    <xacro:include filename="$(find bot_desc)/urdf/mybot/common_inertia.xacro"/>
+    <xacro:macro name ="imu_xacro" params="xyz">
+         <!--机器人的IMU部件and惯性测量传感器-->
+        <link name="imu_link">
+            <visual>
+                <origin xyz="0.0 0.0 0.0" rpy="0.0 0.0 0.0"/>
+                <geometry>
+                    <box size="0.02 0.02 0.02"/>
+                </geometry>
+                <material name="blue">
+                    <color rgba="0.0 0.0 1.0 0.5"/>
+                </material>
+            </visual>
+            <collision>
+                <origin xyz="0.0 0.0 0.0" rpy="0.0 0.0 0.0"/>
+                <geometry>
+                    <box size="0.02 0.02 0.02"/>
+                </geometry>
+                <material name="blue">
+                    <color rgba="0.0 0.0 1.0 0.5"/>
+                </material>
+            </collision>
+            <xacro:box_inertia m="0.05" w="0.02" h="0.02" d="0.02"/>
+        </link>
+        <!--连接身体和IMU的关节-->
+        <joint name="imu_joint" type="fixed">
+            <parent link="base_link"/>
+            <child link="imu_link"/>
+            <origin xyz="${xyz}" rpy="0.0 0.0 0.0"/>
+        </joint>
+            <gazebo reference="imu_link">
+                <material>Gazebo/Blue</material>
+            </gazebo>
+    </xacro:macro>
+</robot>

File: install/bot_desc/share/bot_desc/urdf/mybot/sensor/laser.urdf.xacro (robot description, xacro)
@@ -1 +1,67 @@
-/home/jungle/ros_cpp/robot-/robot-/src/bot_desc/urdf/mybot/sensor/laser.urdf.xacro
+<?xml version="1.0"?>
+<robot xmlns:xacro="http://www.ros.org/wiki/xacro">
+    <xacro:include filename="$(find bot_desc)/urdf/mybot/common_inertia.xacro"/>
+    <xacro:macro name ="laser_xacro" params="xyz">
+    <!--雷达支撑杆-->
+        <link name="laser_cylinder_link">
+            <visual>
+                <origin xyz="0.0 0.0 0.0" rpy="0.0 0.0 0.0"/>
+                <geometry>
+                    <cylinder radius="0.01" length="0.1"/>
+                </geometry>
+                <material name="gray">
+                    <color rgba="0.5 0.5 0.5 1.0"/>
+                </material>
+            </visual>
+            <collision>
+                <origin xyz="0.0 0.0 0.0" rpy="0.0 0.0 0.0"/>
+                <geometry>
+                    <cylinder radius="0.01" length="0.1"/>
+                </geometry>
+                <material name="gray">
+                    <color rgba="0.5 0.5 0.5 1.0"/>
+                </material>
+            </collision>
+            <xacro:cylinder_inertia m="0.05" r="0.01" h="0.1"/>
+        </link>
+         <!--机器人的激光雷达部件-->
+        <link name="laser_link">
+            <visual>
+                <origin xyz="0.0 0.0 0.0" rpy="0.0 0.0 0.0"/>
+                <geometry>
+                    <cylinder radius="0.02" length="0.02"/>
+                </geometry>
+                <material name="red">
+                    <color rgba="1.0 0.0 0.0 0.5"/>
+                </material>
+            </visual>
+            <collision>
+                <origin xyz="0.0 0.0 0.0" rpy="0.0 0.0 0.0"/>
+                <geometry>
+                    <cylinder radius="0.02" length="0.02"/>
+                </geometry>
+                <material name="red">
+                    <color rgba="1.0 0.0 0.0 0.5"/>
+                </material>
+            </collision>
+            <xacro:cylinder_inertia m="0.1" r="0.02" h="0.02"/>
+        </link>
+        <!--连接身体和激光雷达的关节-->
+        <joint name="laser_joint" type="fixed">
+            <parent link="laser_cylinder_link"/>
+            <child link="laser_link"/>
+            <origin xyz="0.0 0.0 0.05" rpy="0.0 0.0 0.0"/>
+        </joint>
+        <joint name="laser_cylinder_joint" type="fixed">
+            <parent link="base_link"/>
+            <child link="laser_cylinder_link"/>
+            <origin xyz="${xyz}" rpy="0.0 0.0 0.0"/>
+        </joint>
+        <gazebo reference="laser_cylinder_link">
+            <material>Gazebo/Black</material>
+        </gazebo>
+        <gazebo reference="laser_link">
+            <material>Gazebo/Black</material>
+        </gazebo>
+    </xacro:macro>
+</robot>

File: src/bot_desc/urdf/mybot/mybot_ros2_control.xacro (robot description, xacro)
@@ -36,4 +36,8 @@
             <plugin filename="libgazebo_ros2_control.so" name="gazebo_ros2_control">
                 <parameters>$(find bot_desc)/config/mybot_ros2_controller.yaml</parameters>
+                <ros>
+                    <remapping>/mybot_diff_drive_controller/odom:=/odom</remapping>
+                    <remapping>/mybot_diff_drive_controller/cmd_vel_unstamped:=/cmd_vel</remapping>
+                </ros>
             </plugin>
         </gazebo>
